File: humidity.sch (KiCad schematic (older format))
At the start: 2 parts, among them U11 SI7020-A10

Commit message: More connections
Parts:
- C21: footprint (none) -> buq2:SM0603
- U11: footprint (none) -> buq2:DFN-6-3X3MM
Changed lines of the file:
@@
 F 0 "U11" H 4600 3050 60  0000 C CNN
 F 1 "SI7020-A10" H 4600 2450 60  0000 C CNN
-F 2 "" H 4550 2600 60  0000 C CNN
+F 2 "buq2:DFN-6-3X3MM" H 4550 2600 60  0001 C CNN
 F 3 "" H 4550 2600 60  0000 C CNN
 	1    4600 2800
@@
 I2C_SDA
 $Comp
-L GND #PWR34
+L GND #PWR036
 U 1 1 5461BC64
 P 4100 2800
-F 0 "#PWR34" H 4100 2800 30  0001 C CNN
+F 0 "#PWR036" H 4100 2800 30  0001 C CNN
 F 1 "GND" H 4100 2730 30  0001 C CNN
 F 2 "" H 4100 2800 60  0000 C CNN
@@
 F 0 "C21" H 5350 3100 40  0000 L CNN
 F 1 "100n" H 5356 2915 40  0000 L CNN
-F 2 "" H 5388 2850 30  0000 C CNN
+F 2 "buq2:SM0603" H 5388 2850 30  0001 C CNN
 F 3 "" H 5350 3000 60  0000 C CNN
 	1    5350 3000
@@
 $EndComp
 $Comp
-L GND #PWR35
+L GND #PWR037
 U 1 1 5461B144
 P 5350 3200
-F 0 "#PWR35" H 5350 3200 30  0001 C CNN
+F 0 "#PWR037" H 5350 3200 30  0001 C CNN
 F 1 "GND" H 5350 3130 30  0001 C CNN
 F 2 "" H 5350 3200 60  0000 C CNN

Commit message: Add buttons. Fix DRC. Add antenna
Parts:
- renumbered U11 to U12, C21 to XC16
Changed lines of the file:
@@
 $Descr A4 11693 8268
 encoding utf-8
-Sheet 12 13
+Sheet 12 14
 Title ""
 Date ""
@@
 $EndDescr
 $Comp
-L SI7020-A10 U11
+L SI7020-A10 U12
 U 1 1 5461BC2E
 P 4600 2800
-F 0 "U11" H 4600 3050 60  0000 C CNN
+F 0 "U12" H 4600 3050 60  0000 C CNN
 F 1 "SI7020-A10" H 4600 2450 60  0000 C CNN
 F 2 "buq2:DFN-6-3X3MM" H 4550 2600 60  0001 C CNN
@@
 I2C_SDA
 $Comp
-L GND #PWR037
+L GND #PWR043
 U 1 1 5461BC64
 P 4100 2800
-F 0 "#PWR037" H 4100 2800 30  0001 C CNN
+F 0 "#PWR043" H 4100 2800 30  0001 C CNN
 F 1 "GND" H 4100 2730 30  0001 C CNN
 F 2 "" H 4100 2800 60  0000 C CNN
@@
 NoConn ~ 5100 2900
 $Comp
-L C C21
+L C XC16
 U 1 1 5461B10D
 P 5350 3000
-F 0 "C21" H 5350 3100 40  0000 L CNN
+F 0 "XC16" H 5350 3100 40  0000 L CNN
 F 1 "100n" H 5356 2915 40  0000 L CNN
 F 2 "buq2:SM0603" H 5388 2850 30  0001 C CNN
@@
 $EndComp
 $Comp
-L GND #PWR038
+L GND #PWR044
 U 1 1 5461B144
 P 5350 3200
-F 0 "#PWR038" H 5350 3200 30  0001 C CNN
+F 0 "#PWR044" H 5350 3200 30  0001 C CNN
 F 1 "GND" H 5350 3130 30  0001 C CNN
 F 2 "" H 5350 3200 60  0000 C CNN
