File: buttons.sch (KiCad schematic (older format))
At the start: 20 parts, among them SW1 SW_LEFT, SW2 SW_DOWN, SW3 SW_UP, SW4 SW_CENTER, SW5 SW_RIGHT

Commit message: Start first layout test
Parts:
- C10, C11, C7, C8, C9, R10, R11, R12, R13, R14, R15, R16, R17, R8, R9: footprint (none) -> buq2:SM0603
- SW1, SW2, SW3, SW4, SW5: footprint (none) -> buq2:PUSHBUTTON_4x4_ROTATED
Changed lines of the file:
@@
 F 0 "SW3" H 5850 2360 50  0000 C CNN
 F 1 "SW_UP" H 5700 2170 50  0000 C CNN
-F 2 "" H 5700 2250 60  0000 C CNN
+F 2 "buq2:PUSHBUTTON_4x4_ROTATED" H 5700 2250 60  0001 C CNN
 F 3 "" H 5700 2250 60  0000 C CNN
 	1    5700 2250
@@
 F 0 "R11" V 6180 1900 40  0000 C CNN
 F 1 "10k" V 6107 1901 40  0000 C CNN
-F 2 "" V 6030 1900 30  0000 C CNN
+F 2 "buq2:SM0603" V 6030 1900 30  0001 C CNN
 F 3 "" H 6100 1900 30  0000 C CNN
 	1    6100 1900
@@
 F 0 "C9" H 6150 2650 40  0000 L CNN
 F 1 "1u" H 6156 2465 40  0000 L CNN
-F 2 "" H 6188 2400 30  0000 C CNN
+F 2 "buq2:SM0603" H 6188 2400 30  0001 C CNN
 F 3 "" H 6150 2550 60  0000 C CNN
 	1    6150 2550
@@
 F 0 "R14" V 6530 2250 40  0000 C CNN
 F 1 "100" V 6457 2251 40  0000 C CNN
-F 2 "" V 6380 2250 30  0000 C CNN
+F 2 "buq2:SM0603" V 6380 2250 30  0001 C CNN
 F 3 "" H 6450 2250 30  0000 C CNN
 	1    6450 2250
@@
 F 0 "SW4" H 5850 3910 50  0000 C CNN
 F 1 "SW_CENTER" H 5700 3720 50  0000 C CNN
-F 2 "" H 5700 3800 60  0000 C CNN
+F 2 "buq2:PUSHBUTTON_4x4_ROTATED" H 5700 3800 60  0001 C CNN
 F 3 "" H 5700 3800 60  0000 C CNN
 	1    5700 3800
@@
 F 0 "R12" V 6180 3450 40  0000 C CNN
 F 1 "10k" V 6107 3451 40  0000 C CNN
-F 2 "" V 6030 3450 30  0000 C CNN
+F 2 "buq2:SM0603" V 6030 3450 30  0001 C CNN
 F 3 "" H 6100 3450 30  0000 C CNN
 	1    6100 3450
@@
 F 0 "C10" H 6150 4200 40  0000 L CNN
 F 1 "1u" H 6156 4015 40  0000 L CNN
-F 2 "" H 6188 3950 30  0000 C CNN
+F 2 "buq2:SM0603" H 6188 3950 30  0001 C CNN
 F 3 "" H 6150 4100 60  0000 C CNN
 	1    6150 4100
@@
 F 0 "R15" V 6530 3800 40  0000 C CNN
 F 1 "100" V 6457 3801 40  0000 C CNN
-F 2 "" V 6380 3800 30  0000 C CNN
+F 2 "buq2:SM0603" V 6380 3800 30  0001 C CNN
 F 3 "" H 6450 3800 30  0000 C CNN
 	1    6450 3800
@@
 F 0 "SW2" H 5800 5410 50  0000 C CNN
 F 1 "SW_DOWN" H 5650 5220 50  0000 C CNN
-F 2 "" H 5650 5300 60  0000 C CNN
+F 2 "buq2:PUSHBUTTON_4x4_ROTATED" H 5650 5300 60  0001 C CNN
 F 3 "" H 5650 5300 60  0000 C CNN
 	1    5650 5300
@@
 F 0 "R10" V 6130 4950 40  0000 C CNN
 F 1 "10k" V 6057 4951 40  0000 C CNN
-F 2 "" V 5980 4950 30  0000 C CNN
+F 2 "buq2:SM0603" V 5980 4950 30  0001 C CNN
 F 3 "" H 6050 4950 30  0000 C CNN
 	1    6050 4950
@@
 F 0 "C8" H 6100 5700 40  0000 L CNN
 F 1 "1u" H 6106 5515 40  0000 L CNN
-F 2 "" H 6138 5450 30  0000 C CNN
+F 2 "buq2:SM0603" H 6138 5450 30  0001 C CNN
 F 3 "" H 6100 5600 60  0000 C CNN
 	1    6100 5600
@@
 F 0 "R13" V 6480 5300 40  0000 C CNN
 F 1 "100" V 6407 5301 40  0000 C CNN
-F 2 "" V 6330 5300 30  0000 C CNN
+F 2 "buq2:SM0603" V 6330 5300 30  0001 C CNN
 F 3 "" H 6400 5300 30  0000 C CNN
 	1    6400 5300
@@
 F 0 "SW1" H 3450 3910 50  0000 C CNN
 F 1 "SW_LEFT" H 3300 3720 50  0000 C CNN
-F 2 "" H 3300 3800 60  0000 C CNN
+F 2 "buq2:PUSHBUTTON_4x4_ROTATED" H 3300 3800 60  0001 C CNN
 F 3 "" H 3300 3800 60  0000 C CNN
 	1    3300 3800
@@
 F 0 "R8" V 3780 3450 40  0000 C CNN
 F 1 "10k" V 3707 3451 40  0000 C CNN
-F 2 "" V 3630 3450 30  0000 C CNN
+F 2 "buq2:SM0603" V 3630 3450 30  0001 C CNN
 F 3 "" H 3700 3450 30  0000 C CNN
 	1    3700 3450
@@
 F 0 "C7" H 3750 4200 40  0000 L CNN
 F 1 "1u" H 3756 4015 40  0000 L CNN
-F 2 "" H 3788 3950 30  0000 C CNN
+F 2 "buq2:SM0603" H 3788 3950 30  0001 C CNN
 F 3 "" H 3750 4100 60  0000 C CNN
 	1    3750 4100
@@
 F 0 "R9" V 4130 3800 40  0000 C CNN
 F 1 "100" V 4057 3801 40  0000 C CNN
-F 2 "" V 3980 3800 30  0000 C CNN
+F 2 "buq2:SM0603" V 3980 3800 30  0001 C CNN
 F 3 "" H 4050 3800 30  0000 C CNN
 	1    4050 3800
@@
 F 0 "SW5" H 8250 3860 50  0000 C CNN
 F 1 "SW_RIGHT" H 8100 3670 50  0000 C CNN
-F 2 "" H 8100 3750 60  0000 C CNN
+F 2 "buq2:PUSHBUTTON_4x4_ROTATED" H 8100 3750 60  0001 C CNN
 F 3 "" H 8100 3750 60  0000 C CNN
 	1    8100 3750
@@
 F 0 "R16" V 8580 3400 40  0000 C CNN
 F 1 "10k" V 8507 3401 40  0000 C CNN
-F 2 "" V 8430 3400 30  0000 C CNN
+F 2 "buq2:SM0603" V 8430 3400 30  0001 C CNN
 F 3 "" H 8500 3400 30  0000 C CNN
 	1    8500 3400
@@
 F 0 "C11" H 8550 4150 40  0000 L CNN
 F 1 "1u" H 8556 3965 40  0000 L CNN
-F 2 "" H 8588 3900 30  0000 C CNN
+F 2 "buq2:SM0603" H 8588 3900 30  0001 C CNN
 F 3 "" H 8550 4050 60  0000 C CNN
 	1    8550 4050
@@
 F 0 "R17" V 8930 3750 40  0000 C CNN
 F 1 "100" V 8857 3751 40  0000 C CNN
-F 2 "" V 8780 3750 30  0000 C CNN
+F 2 "buq2:SM0603" V 8780 3750 30  0001 C CNN
 F 3 "" H 8850 3750 30  0000 C CNN
 	1    8850 3750

Commit message: Before adding proper reset and battery monitor
Parts:
- SW1, SW2, SW3, SW4, SW5: footprint buq2:PUSHBUTTON_4x4_ROTATED -> buq2:PUSHBUTTON_4x4_5x5_ROTATED
Changed lines of the file:
@@
 F 0 "SW3" H 5850 2360 50  0000 C CNN
 F 1 "SW_UP" H 5700 2170 50  0000 C CNN
-F 2 "buq2:PUSHBUTTON_4x4_ROTATED" H 5700 2250 60  0001 C CNN
+F 2 "buq2:PUSHBUTTON_4x4_5x5_ROTATED" H 5700 2250 60  0001 C CNN
 F 3 "" H 5700 2250 60  0000 C CNN
 	1    5700 2250
@@
 F 0 "SW4" H 5850 3910 50  0000 C CNN
 F 1 "SW_CENTER" H 5700 3720 50  0000 C CNN
-F 2 "buq2:PUSHBUTTON_4x4_ROTATED" H 5700 3800 60  0001 C CNN
+F 2 "buq2:PUSHBUTTON_4x4_5x5_ROTATED" H 5700 3800 60  0001 C CNN
 F 3 "" H 5700 3800 60  0000 C CNN
 	1    5700 3800
@@
 F 0 "SW2" H 5800 5410 50  0000 C CNN
 F 1 "SW_DOWN" H 5650 5220 50  0000 C CNN
-F 2 "buq2:PUSHBUTTON_4x4_ROTATED" H 5650 5300 60  0001 C CNN
+F 2 "buq2:PUSHBUTTON_4x4_5x5_ROTATED" H 5650 5300 60  0001 C CNN
 F 3 "" H 5650 5300 60  0000 C CNN
 	1    5650 5300
@@
 F 0 "SW1" H 3450 3910 50  0000 C CNN
 F 1 "SW_LEFT" H 3300 3720 50  0000 C CNN
-F 2 "buq2:PUSHBUTTON_4x4_ROTATED" H 3300 3800 60  0001 C CNN
+F 2 "buq2:PUSHBUTTON_4x4_5x5_ROTATED" H 3300 3800 60  0001 C CNN
 F 3 "" H 3300 3800 60  0000 C CNN
 	1    3300 3800
@@
 F 0 "SW5" H 8250 3860 50  0000 C CNN
 F 1 "SW_RIGHT" H 8100 3670 50  0000 C CNN
-F 2 "buq2:PUSHBUTTON_4x4_ROTATED" H 8100 3750 60  0001 C CNN
+F 2 "buq2:PUSHBUTTON_4x4_5x5_ROTATED" H 8100 3750 60  0001 C CNN
 F 3 "" H 8100 3750 60  0000 C CNN
 	1    8100 3750

Commit message: Start planning test board v2.0
Parts:
- removed C10, C11, C7, C8, C9: 1u, buq2:SM0603, symbol C
- removed R10, R11, R12, R16, R8: 10k, buq2:SM0603, symbol R
- removed R13, R14, R15, R17, R9: 100, buq2:SM0603, symbol R
- removed SW1: SW_LEFT, buq2:PUSHBUTTON_4x4_5x5_ROTATED, symbol SW_PUSH
- removed SW2: SW_DOWN, buq2:PUSHBUTTON_4x4_5x5_ROTATED, symbol SW_PUSH
- removed SW3: SW_UP, buq2:PUSHBUTTON_4x4_5x5_ROTATED, symbol SW_PUSH
- removed SW4: SW_CENTER, buq2:PUSHBUTTON_4x4_5x5_ROTATED, symbol SW_PUSH
- removed SW5: SW_RIGHT, buq2:PUSHBUTTON_4x4_5x5_ROTATED, symbol SW_PUSH
- added U10: CNT, buq2:PUSHBUTTON_4x4_5x5_ROTATED_4_PIN, symbol SW_PUSH_4_PIN
- added U11: DWN, buq2:PUSHBUTTON_4x4_5x5_ROTATED_4_PIN, symbol SW_PUSH_4_PIN
- added U4: UP, buq2:PUSHBUTTON_4x4_5x5_ROTATED_4_PIN, symbol SW_PUSH_4_PIN
Connections:
- net labels removed: BUTTON_LEFT, BUTTON_RIGHT, VDD
- wire segments 30 -> 6
- no-connect marks 0 -> 6
