File: clock.sch (KiCad schematic (older format))
At the start: 5 parts, among them U1 MCP7940M, X1 CRYSTAL

Commit message: Add gps
Parts:
- added R3: 10k, symbol R
Connections:
- net GND: now also U1.4 (Vss)
- net I2C_SDA: now reaches U1.5 (SDA)
- net I2C_SCL: now reaches U1.6 (SCL)
- net MULTI_FUNCTIONAL: now reaches U1.7 (MFP)
- net MULTI_FUNCTIONAL: now also R3.2
- net VCC: now reaches C3.2, U1.8 (Vcc)
- net VCC: now also R3.1
Changed lines of the file:
@@
 $Descr A4 11693 8268
 encoding utf-8
-Sheet 2 10
+Sheet 2 11
 Title ""
 Date ""
@@
 $EndComp
 $Comp
-L GND #PWR2
+L GND #PWR3
 U 1 1 54461061
 P 4550 1650
-F 0 "#PWR2" H 4550 1650 30  0001 C CNN
+F 0 "#PWR3" H 4550 1650 30  0001 C CNN
 F 1 "GND" H 4550 1580 30  0001 C CNN
 F 2 "" H 4550 1650 60  0000 C CNN
@@
 	4550 1650 4550 1750
 Wire Wire Line
-	4550 2150 4450 2150
+	4950 2150 4450 2150
+Text HLabel 4450 2450 2    60   Input ~ 0
+I2C_SCL
+Text HLabel 4450 2600 2    60   Input ~ 0
+I2C_SDA
+$Comp
+L GND #PWR2
+U 1 1 5460FDF5
+P 3450 2600
+F 0 "#PWR2" H 3450 2600 30  0001 C CNN
+F 1 "GND" H 3450 2530 30  0001 C CNN
+F 2 "" H 3450 2600 60  0000 C CNN
+F 3 "" H 3450 2600 60  0000 C CNN
+	1    3450 2600
+	0    1    1    0
+$EndComp
+Text HLabel 4950 1650 1    60   Input ~ 0
+VCC
+$Comp
+L R R3
+U 1 1 5460FE77
+P 5050 2050
+F 0 "R3" V 5130 2050 40  0000 C CNN
+F 1 "10k" V 5057 2051 40  0000 C CNN
+F 2 "" V 4980 2050 30  0000 C CNN
+F 3 "" H 5050 2050 30  0000 C CNN
+	1    5050 2050
+	1    0    0    -1
+$EndComp
+Wire Wire Line
+	4450 2300 5050 2300
+Text HLabel 5050 2300 2    60   Input ~ 0
+MULTI_FUNCTIONAL
+Wire Wire Line
+	5050 1800 4950 1800
+Wire Wire Line
+	4950 1650 4950 2150
+Connection ~ 4550 2150
+Connection ~ 4950 1800
 $EndSCHEMATC

Commit message: More connections
Parts:
- C1, C2, C3, R3: footprint (none) -> buq2:SM0603
- U1: footprint (none) -> buq2:8-SOIC
- X1: footprint (none) -> buq2:SM0805
Changed lines of the file:
@@
 F 0 "U1" H 3950 2200 60  0000 C CNN
 F 1 "MCP7940M" H 3950 3200 60  0000 C CNN
-F 2 "" H 4000 2550 60  0001 C CNN
+F 2 "buq2:8-SOIC" H 4000 2550 60  0001 C CNN
 F 3 "" H 4000 2550 60  0000 C CNN
 	1    4000 2550
@@
 F 0 "X1" H 3000 2400 60  0000 C CNN
 F 1 "CRYSTAL" H 3000 2100 60  0000 C CNN
-F 2 "" H 3000 2250 60  0001 C CNN
+F 2 "buq2:SM0805" H 3000 2250 60  0001 C CNN
 F 3 "" H 3000 2250 60  0000 C CNN
 	1    3000 2250
@@
 F 0 "C1" H 2800 2050 40  0000 L CNN
 F 1 "C" H 2806 1865 40  0000 L CNN
-F 2 "" H 2838 1800 30  0001 C CNN
+F 2 "buq2:SM0603" H 2838 1800 30  0001 C CNN
 F 3 "" H 2800 1950 60  0000 C CNN
 	1    2800 1950
@@
 F 0 "C2" H 2800 2650 40  0000 L CNN
 F 1 "C" H 2806 2465 40  0000 L CNN
-F 2 "" H 2838 2400 30  0001 C CNN
+F 2 "buq2:SM0603" H 2838 2400 30  0001 C CNN
 F 3 "" H 2800 2550 60  0000 C CNN
 	1    2800 2550
@@
 $EndComp
 $Comp
-L GND #PWR1
+L GND #PWR01
 U 1 1 54461054
 P 2500 2250
-F 0 "#PWR1" H 2500 2250 30  0001 C CNN
+F 0 "#PWR01" H 2500 2250 30  0001 C CNN
 F 1 "GND" H 2500 2180 30  0001 C CNN
 F 2 "" H 2500 2250 60  0000 C CNN
@@
 F 0 "C3" H 4550 2050 40  0000 L CNN
 F 1 "100n" H 4556 1865 40  0000 L CNN
-F 2 "" H 4588 1800 30  0001 C CNN
+F 2 "buq2:SM0603" H 4588 1800 30  0001 C CNN
 F 3 "" H 4550 1950 60  0000 C CNN
 	1    4550 1950
@@
 $EndComp
 $Comp
-L GND #PWR3
+L GND #PWR02
 U 1 1 54461061
 P 4550 1650
-F 0 "#PWR3" H 4550 1650 30  0001 C CNN
+F 0 "#PWR02" H 4550 1650 30  0001 C CNN
 F 1 "GND" H 4550 1580 30  0001 C CNN
 F 2 "" H 4550 1650 60  0000 C CNN
@@
 I2C_SDA
 $Comp
-L GND #PWR2
+L GND #PWR03
 U 1 1 5460FDF5
 P 3450 2600
-F 0 "#PWR2" H 3450 2600 30  0001 C CNN
+F 0 "#PWR03" H 3450 2600 30  0001 C CNN
 F 1 "GND" H 3450 2530 30  0001 C CNN
 F 2 "" H 3450 2600 60  0000 C CNN
@@
 F 0 "R3" V 5130 2050 40  0000 C CNN
 F 1 "10k" V 5057 2051 40  0000 C CNN
-F 2 "" V 4980 2050 30  0000 C CNN
+F 2 "buq2:SM0603" V 4980 2050 30  0001 C CNN
 F 3 "" H 5050 2050 30  0000 C CNN
 	1    5050 2050

Commit message: Add buttons. Fix DRC. Add antenna
Parts:
- C1, C2: value C -> 18.1p
- renumbered R3 to R1, C3 to XC1
Changed lines of the file:
@@
 $Descr A4 11693 8268
 encoding utf-8
-Sheet 2 13
+Sheet 2 14
 Title ""
 Date ""
@@
 P 2800 1950
 F 0 "C1" H 2800 2050 40  0000 L CNN
-F 1 "C" H 2806 1865 40  0000 L CNN
+F 1 "18.1p" H 2806 1865 40  0000 L CNN
 F 2 "buq2:SM0603" H 2838 1800 30  0001 C CNN
 F 3 "" H 2800 1950 60  0000 C CNN
@@
 P 2800 2550
 F 0 "C2" H 2800 2650 40  0000 L CNN
-F 1 "C" H 2806 2465 40  0000 L CNN
+F 1 "18.1p" H 2806 2465 40  0000 L CNN
 F 2 "buq2:SM0603" H 2838 2400 30  0001 C CNN
 F 3 "" H 2800 2550 60  0000 C CNN
@@
 $EndComp
 $Comp
-L C C3
+L C XC1
 U 1 1 5446105A
 P 4550 1950
-F 0 "C3" H 4550 2050 40  0000 L CNN
+F 0 "XC1" H 4550 2050 40  0000 L CNN
 F 1 "100n" H 4556 1865 40  0000 L CNN
 F 2 "buq2:SM0603" H 4588 1800 30  0001 C CNN
@@
 VCC
 $Comp
-L R R3
+L R R1
 U 1 1 5460FE77
 P 5050 2050
-F 0 "R3" V 5130 2050 40  0000 C CNN
+F 0 "R1" V 5130 2050 40  0000 C CNN
 F 1 "10k" V 5057 2051 40  0000 C CNN
 F 2 "buq2:SM0603" V 4980 2050 30  0001 C CNN

Commit message: Start first layout test
Parts:
- U1: footprint buq2:8-SOIC -> buq2:8-TDFN
Changed lines of the file:
@@
 F 0 "U1" H 3950 2200 60  0000 C CNN
 F 1 "MCP7940M" H 3950 3200 60  0000 C CNN
-F 2 "buq2:8-SOIC" H 4000 2550 60  0001 C CNN
+F 2 "buq2:8-TDFN" H 4000 2550 60  0001 C CNN
 F 3 "" H 4000 2550 60  0000 C CNN
 	1    4000 2550
