File: mcu.sch (KiCad schematic (older format))
At the start: 10 parts, among them IC1 BUQ2-ATXMEGA128A4U-A, U9 TAG-CONNECT-ATMEL-PDI-CONNECT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

Commit message: Start planning test board v2.0
Parts:
- removed R20, R21: 10k, buq2:SM0603, symbol R
Connections:
- net BUTTON_LEFT is gone; now on net BUTTON_CENTER: IC1.2 (AC1OUT/AC6/ADC6/PA6)
- net CSn_RAM is gone; now on net CSp_DISPLAY: IC1.21 (PD1/OC0B/XCK0)
- net BUTTON_CENTER: no longer IC1.3 (AC0OUT/AC7/ADC7/PA7)
- net BUTTON_DOWN: now also IC1.3 (AC0OUT/AC7/ADC7/PA7); no longer IC1.5 (ADC9/PB1)
- net BUZZER_DRIVE: now also IC1.24 (PD4/OC1A/~SS~); no longer IC1.7 (DAC1/ACD11/PB3)
- net CSp_DISPLAY: no longer IC1.22 (PD2/OC0C/RXD0)
- net ACCELERATOR_INT: no longer names the net of IC1.41 (AC1/ADC1/PA1)
- net BUTTON_RIGHT: no longer names the net of IC1.4 (AREFB/ADC8/PB0)
- net CSn_SD_CARD: no longer names the net of IC1.23 (PD3/OC0D/TXD0)
- net DISPLAY_INVERT: no longer names the net of IC1.6 (DAC0/ADC10/PB2)
- net GPS_PULSE_PER_SECOND: no longer names the net of IC1.44 (AC4/ADC4/PA4)
- net RX: no longer names the net of IC1.32 (PE2/OC0C/RXD0)
- net SD_CARD_DETECT: no longer names the net of IC1.43 (AC3/ADC3/PA3)
- net TX: no longer names the net of IC1.33 (PE3/OC0D/TXD0)
- new net DISP_ON: IC1.22 (PD2/OC0C/RXD0)
- no-connect marks 11 -> 20
Other:
- note removed: "These pull-up/downs\nare only for possible\ndebugging.\nRemove from final."
Changed lines of the file:
@@
 $Descr A4 11693 8268
 encoding utf-8
-Sheet 9 14
+Sheet 8 10
 Title ""
 Date ""
@@
 Text Notes 2550 4500 0    60   ~ 0
 USB
-Text HLabel 3000 3550 0    60   Input ~ 0
-RX
-Text HLabel 3000 3650 0    60   Input ~ 0
-TX
 $Comp
 L R R5
@@
 Text Label 3000 2600 2    60   ~ 0
 PDI_DATA
-Text HLabel 5700 3550 2    60   Input ~ 0
-DISPLAY_INVERT
-Text HLabel 5700 3650 2    60   Input ~ 0
+Text HLabel 3000 4200 0    60   Input ~ 0
 BUZZER_DRIVE
 Text HLabel 5700 2500 2    60   Input ~ 0
 CLOCK_INT
-Text HLabel 5700 2600 2    60   Input ~ 0
-ACCELERATOR_INT
 Text HLabel 5700 2700 2    60   Input ~ 0
 BAROMETER_INT
@@
 CSn_FLASH
 Text HLabel 3000 3900 0    60   Input ~ 0
-CSn_RAM
-Text HLabel 3000 4000 0    60   Input ~ 0
 CSp_DISPLAY
-Text HLabel 3000 4100 0    60   Input ~ 0
-CSn_SD_CARD
-Text HLabel 5700 2800 2    60   Input ~ 0
-SD_CARD_DETECT
 NoConn ~ 3000 4300
 NoConn ~ 3000 3450
@@
 NoConn ~ 5700 4100
 NoConn ~ 5700 4200
-NoConn ~ 3000 4200
-Text HLabel 5700 2900 2    60   Input ~ 0
-GPS_PULSE_PER_SECOND
 Text HLabel 5700 3000 2    60   Input ~ 0
 BUTTON_UP
-Text HLabel 5700 3450 2    60   Input ~ 0
+Text HLabel 5700 3200 2    60   Input ~ 0
 BUTTON_DOWN
 Text HLabel 5700 3100 2    60   Input ~ 0
-BUTTON_LEFT
-Text HLabel 5700 3350 2    60   Input ~ 0
-BUTTON_RIGHT
-Text HLabel 5700 3200 2    60   Input ~ 0
 BUTTON_CENTER
-$Comp
-L R R20
-U 1 1 547A08E0
-P 7050 4150
-F 0 "R20" V 7130 4150 40  0000 C CNN
-F 1 "10k" V 7057 4151 40  0000 C CNN
-F 2 "buq2:SM0603" V 6980 4150 30  0001 C CNN
-F 3 "" H 7050 4150 30  0000 C CNN
-	1    7050 4150
-	1    0    0    -1
-$EndComp
-$Comp
-L R R21
-U 1 1 547A090C
-P 7050 4650
-F 0 "R21" V 7130 4650 40  0000 C CNN
-F 1 "10k" V 7057 4651 40  0000 C CNN
-F 2 "buq2:SM0603" V 6980 4650 30  0001 C CNN
-F 3 "" H 7050 4650 30  0000 C CNN
-	1    7050 4650
-	1    0    0    -1
-$EndComp
-$Comp
-L GND #PWR028
-U 1 1 547A0947
-P 7050 4900
-F 0 "#PWR028" H 7050 4900 30  0001 C CNN
-F 1 "GND" H 7050 4830 30  0001 C CNN
-F 2 "" H 7050 4900 60  0000 C CNN
-F 3 "" H 7050 4900 60  0000 C CNN
-	1    7050 4900
-	1    0    0    -1
-$EndComp
-Text HLabel 7050 3900 1    60   Input ~ 0
-VDD
 Wire Wire Line
 	5700 4400 7250 4400
 Connection ~ 7050 4400
-Text Notes 7200 4800 0    60   ~ 0
-These pull-up/downs\nare only for possible\ndebugging.\nRemove from final.
+NoConn ~ 3000 3550
+NoConn ~ 3000 3650
+NoConn ~ 3000 4100
+NoConn ~ 5700 3350
+Text HLabel 3000 4000 0    60   Input ~ 0
+DISP_ON
+NoConn ~ 5700 2600
+NoConn ~ 5700 2800
+NoConn ~ 5700 2900
+NoConn ~ 5700 3450
+NoConn ~ 5700 3550
+NoConn ~ 5700 3650
 $EndSCHEMATC

Commit message: Almost ready routing
Connections:
- net BAROMETER_INT: now also IC1.7 (DAC1/ACD11/PB3); no longer IC1.42 (AC2/ADC2/PA2)
- net BUTTON_CENTER: now also IC1.13 (SCLOUT/TXD0/OC0BHS/OC0D/PC3); no longer IC1.2 (AC1OUT/AC6/ADC6/PA6)
- net BUTTON_DOWN: now also IC1.12 (SDAOUT/RXD0/~OC0BLS~/OC0C/PC2); no longer IC1.3 (AC0OUT/AC7/ADC7/PA7)
- net BUTTON_UP: now also IC1.14 (~SS~/~OC0CLS~/OC1A/PC4); no longer IC1.1 (AC5/ADC5/PA5)
- net CLOCK_INT: now also IC1.6 (DAC0/ADC10/PB2); no longer IC1.40 (AREFA/AC0/ADC0/PA0)
- net CSn_FLASH: now also IC1.44 (AC4/ADC4/PA4); no longer IC1.20 (PD0/OC0A)
- net CSp_DISPLAY: now also IC1.43 (AC3/ADC3/PA3); no longer IC1.21 (PD1/OC0B/XCK0)
- net DISP_ON: now also IC1.42 (AC2/ADC2/PA2); no longer IC1.22 (PD2/OC0C/RXD0)
Changed lines of the file:
@@
 Text HLabel 5700 4300 2    60   Input ~ 0
 MOSI
-Text HLabel 7250 4400 2    60   Input ~ 0
+Text HLabel 5700 4400 2    60   Input ~ 0
 MISO
 Text HLabel 5700 4500 2    60   Input ~ 0
@@
 Text HLabel 3000 4200 0    60   Input ~ 0
 BUZZER_DRIVE
-Text HLabel 5700 2500 2    60   Input ~ 0
+Text HLabel 5700 3550 2    60   Input ~ 0
 CLOCK_INT
-Text HLabel 5700 2700 2    60   Input ~ 0
+Text HLabel 5700 3650 2    60   Input ~ 0
 BAROMETER_INT
-Text HLabel 3000 3800 0    60   Input ~ 0
+Text HLabel 5700 2900 2    60   Input ~ 0
 CSn_FLASH
-Text HLabel 3000 3900 0    60   Input ~ 0
+Text HLabel 5700 2800 2    60   Input ~ 0
 CSp_DISPLAY
 NoConn ~ 3000 4300
@@
 NoConn ~ 3000 3200
 NoConn ~ 3000 3100
-NoConn ~ 5700 4000
-NoConn ~ 5700 4100
-NoConn ~ 5700 4200
-Text HLabel 5700 3000 2    60   Input ~ 0
+NoConn ~ 5700 3000
+NoConn ~ 5700 3100
+NoConn ~ 5700 3200
+Text HLabel 5700 4200 2    60   Input ~ 0
 BUTTON_UP
-Text HLabel 5700 3200 2    60   Input ~ 0
+Text HLabel 5700 4000 2    60   Input ~ 0
 BUTTON_DOWN
-Text HLabel 5700 3100 2    60   Input ~ 0
+Text HLabel 5700 4100 2    60   Input ~ 0
 BUTTON_CENTER
-Wire Wire Line
-	5700 4400 7250 4400
-Connection ~ 7050 4400
 NoConn ~ 3000 3550
 NoConn ~ 3000 3650
 NoConn ~ 3000 4100
 NoConn ~ 5700 3350
-Text HLabel 3000 4000 0    60   Input ~ 0
+Text HLabel 5700 2700 2    60   Input ~ 0
 DISP_ON
 NoConn ~ 5700 2600
-NoConn ~ 5700 2800
-NoConn ~ 5700 2900
+NoConn ~ 3000 4000
+NoConn ~ 3000 3900
 NoConn ~ 5700 3450
-NoConn ~ 5700 3550
-NoConn ~ 5700 3650
+NoConn ~ 3000 3800
+NoConn ~ 5700 2500
 $EndSCHEMATC

Commit message: Ordered version 2.0 (pcb and stencil)
Parts:
- added P2: SERIAL, buq2:PIN_HEADER_2, symbol CONN_2
Connections:
- net at IC1.32 (PE2/OC0C/RXD0): now also P2.2 (PM)
- net at IC1.33 (PE3/OC0D/TXD0): now also P2.1 (P1)
- no-connect marks 20 -> 18
Changed lines of the file:
@@
 $EndComp
 $Comp
-L GND #PWR27
+L GND #PWR028
 U 1 1 54464F33
 P 4100 1400
-F 0 "#PWR27" H 4100 1400 30  0001 C CNN
+F 0 "#PWR028" H 4100 1400 30  0001 C CNN
 F 1 "GND" H 4100 1330 30  0001 C CNN
 F 2 "" H 4100 1400 60  0000 C CNN
@@
 NoConn ~ 6100 1450
 $Comp
-L GND #PWR28
+L GND #PWR029
 U 1 1 54464F41
 P 7250 1600
-F 0 "#PWR28" H 7250 1600 30  0001 C CNN
+F 0 "#PWR029" H 7250 1600 30  0001 C CNN
 F 1 "GND" H 7250 1530 30  0001 C CNN
 F 2 "" H 7250 1600 60  0000 C CNN
@@
 $EndComp
 $Comp
-L GND #PWR26
+L GND #PWR030
 U 1 1 54464F47
 P 3900 5100
-F 0 "#PWR26" H 3900 5100 30  0001 C CNN
+F 0 "#PWR030" H 3900 5100 30  0001 C CNN
 F 1 "GND" H 3900 5030 30  0001 C CNN
 F 2 "" H 3900 5100 60  0000 C CNN
@@
 Text HLabel 5700 4100 2    60   Input ~ 0
 BUTTON_CENTER
-NoConn ~ 3000 3550
-NoConn ~ 3000 3650
 NoConn ~ 3000 4100
 NoConn ~ 5700 3350
@@
 NoConn ~ 3000 3800
 NoConn ~ 5700 2500
+$Comp
+L CONN_2 P2
+U 1 1 54C7F3AD
+P 1550 3400
+F 0 "P2" V 1500 3400 40  0000 C CNN
+F 1 "SERIAL" V 1600 3400 40  0000 C CNN
+F 2 "buq2:PIN_HEADER_2" H 1550 3400 60  0001 C CNN
+F 3 "" H 1550 3400 60  0000 C CNN
+	1    1550 3400
+	-1   0    0    1
+$EndComp
+Wire Wire Line
+	3000 3550 2400 3550
+Wire Wire Line
+	2400 3550 2400 3300
+Wire Wire Line
+	2400 3300 1900 3300
+Wire Wire Line
+	3000 3650 1900 3650
+Wire Wire Line
+	1900 3650 1900 3500
 $EndSCHEMATC

Commit message: Start implementing new version: move USB port and altimeter module, new buzzer and volume control
Connections:
- net BUTTON_CENTER: now also IC1.2 (AC1OUT/AC6/ADC6/PA6); no longer IC1.13 (SCLOUT/TXD0/OC0BHS/OC0D/PC3)
- net BUTTON_DOWN: now also IC1.1 (AC5/ADC5/PA5); no longer IC1.12 (SDAOUT/RXD0/~OC0BLS~/OC0C/PC2)
- net BUTTON_UP: now also IC1.3 (AC0OUT/AC7/ADC7/PA7); no longer IC1.14 (~SS~/~OC0CLS~/OC1A/PC4)
Changed lines of the file:
@@
 $EndComp
 $Comp
-L GND #PWR028
+L GND #PWR030
 U 1 1 54464F33
 P 4100 1400
-F 0 "#PWR028" H 4100 1400 30  0001 C CNN
+F 0 "#PWR030" H 4100 1400 30  0001 C CNN
 F 1 "GND" H 4100 1330 30  0001 C CNN
 F 2 "" H 4100 1400 60  0000 C CNN
@@
 NoConn ~ 6100 1450
 $Comp
-L GND #PWR029
+L GND #PWR031
 U 1 1 54464F41
 P 7250 1600
-F 0 "#PWR029" H 7250 1600 30  0001 C CNN
+F 0 "#PWR031" H 7250 1600 30  0001 C CNN
 F 1 "GND" H 7250 1530 30  0001 C CNN
 F 2 "" H 7250 1600 60  0000 C CNN
@@
 $EndComp
 $Comp
-L GND #PWR030
+L GND #PWR032
 U 1 1 54464F47
 P 3900 5100
-F 0 "#PWR030" H 3900 5100 30  0001 C CNN
+F 0 "#PWR032" H 3900 5100 30  0001 C CNN
 F 1 "GND" H 3900 5030 30  0001 C CNN
 F 2 "" H 3900 5100 60  0000 C CNN
@@
 NoConn ~ 3000 3200
 NoConn ~ 3000 3100
-NoConn ~ 5700 3000
-NoConn ~ 5700 3100
-NoConn ~ 5700 3200
-Text HLabel 5700 4200 2    60   Input ~ 0
+NoConn ~ 5700 4000
+NoConn ~ 5700 4100
+NoConn ~ 5700 4200
+Text HLabel 5700 3200 2    60   Input ~ 0
 BUTTON_UP
-Text HLabel 5700 4000 2    60   Input ~ 0
+Text HLabel 5700 3000 2    60   Input ~ 0
 BUTTON_DOWN
-Text HLabel 5700 4100 2    60   Input ~ 0
+Text HLabel 5700 3100 2    60   Input ~ 0
 BUTTON_CENTER
 NoConn ~ 3000 4100

Commit message: Before starting laying out tracks
Parts:
- added P3: POWER, buq2:PIN_HEADER_2, symbol CONN_2
Connections:
- net GND: now also P3.1 (P1)
- net VDD: now also IC1.40 (AREFA/AC0/ADC0/PA0), P3.2 (PM)
- net ACC_INT: now reaches IC1.5 (ADC9/PB1)
- no-connect marks 18 -> 16
Other:
- note added: "VDD at AREF should make it possible for simple battery monitor"
Changed lines of the file:
@@
 $Descr A4 11693 8268
 encoding utf-8
-Sheet 8 10
+Sheet 8 11
 Title ""
 Date ""
@@
 NoConn ~ 3000 4000
 NoConn ~ 3000 3900
-NoConn ~ 5700 3450
 NoConn ~ 3000 3800
-NoConn ~ 5700 2500
 $Comp
 L CONN_2 P2
@@
 Wire Wire Line
 	1900 3650 1900 3500
+$Comp
+L CONN_2 P3
+U 1 1 552F44E9
+P 1550 3950
+F 0 "P3" V 1500 3950 40  0000 C CNN
+F 1 "POWER" V 1600 3950 40  0000 C CNN
+F 2 "buq2:PIN_HEADER_2" H 1550 3950 60  0001 C CNN
+F 3 "" H 1550 3950 60  0000 C CNN
+	1    1550 3950
+	-1   0    0    1
+$EndComp
+Text HLabel 1900 3850 2    60   Input ~ 0
+VDD
+$Comp
+L GND #PWR033
+U 1 1 552F45D9
+P 1950 4050
+F 0 "#PWR033" H 1950 4050 30  0001 C CNN
+F 1 "GND" H 1950 3980 30  0001 C CNN
+F 2 "" H 1950 4050 60  0000 C CNN
+F 3 "" H 1950 4050 60  0000 C CNN
+	1    1950 4050
+	0    -1   -1   0
+$EndComp
+Wire Wire Line
+	1950 4050 1900 4050
+Text HLabel 5700 2500 2    60   Input ~ 0
+VDD
+Text Notes 5600 2200 0    60   ~ 0
+VDD at AREF should make it possible for simple battery monitor
+Text HLabel 5700 3450 2    60   Input ~ 0
+ACC_INT
 $EndSCHEMATC

Commit message: Ordered v3.0
Connections:
- net BUTTON_CENTER: now also IC1.21 (PD1/OC0B/XCK0); no longer IC1.2 (AC1OUT/AC6/ADC6/PA6)
- net BUTTON_DOWN: now also IC1.20 (PD0/OC0A); no longer IC1.1 (AC5/ADC5/PA5)
- net BUTTON_UP: now also IC1.22 (PD2/OC0C/RXD0); no longer IC1.3 (AC0OUT/AC7/ADC7/PA7)
- net RX: now reaches IC1.32 (PE2/OC0C/RXD0)
- net RX: now also P2.1 (P1); no longer P2.2 (PM)
- net TX: now reaches IC1.33 (PE3/OC0D/TXD0)
- net TX: now also P2.2 (PM); no longer P2.1 (P1)
Changed lines of the file:
@@
 $EndComp
 $Comp
-L GND #PWR30
+L GND #PWR030
 U 1 1 54464F33
 P 4100 1400
-F 0 "#PWR30" H 4100 1400 30  0001 C CNN
+F 0 "#PWR030" H 4100 1400 30  0001 C CNN
 F 1 "GND" H 4100 1330 30  0001 C CNN
 F 2 "" H 4100 1400 60  0000 C CNN
@@
 NoConn ~ 6100 1450
 $Comp
-L GND #PWR31
+L GND #PWR031
 U 1 1 54464F41
 P 7250 1600
-F 0 "#PWR31" H 7250 1600 30  0001 C CNN
+F 0 "#PWR031" H 7250 1600 30  0001 C CNN
 F 1 "GND" H 7250 1530 30  0001 C CNN
 F 2 "" H 7250 1600 60  0000 C CNN
@@
 $EndComp
 $Comp
-L GND #PWR29
+L GND #PWR032
 U 1 1 54464F47
 P 3900 5100
-F 0 "#PWR29" H 3900 5100 30  0001 C CNN
+F 0 "#PWR032" H 3900 5100 30  0001 C CNN
 F 1 "GND" H 3900 5030 30  0001 C CNN
 F 2 "" H 3900 5100 60  0000 C CNN
@@
 NoConn ~ 5700 4100
 NoConn ~ 5700 4200
-Text HLabel 5700 3200 2    60   Input ~ 0
+Text HLabel 3000 4000 0    60   Input ~ 0
 BUTTON_UP
-Text HLabel 5700 3000 2    60   Input ~ 0
+Text HLabel 3000 3800 0    60   Input ~ 0
 BUTTON_DOWN
-Text HLabel 5700 3100 2    60   Input ~ 0
+Text HLabel 3000 3900 0    60   Input ~ 0
 BUTTON_CENTER
 NoConn ~ 3000 4100
@@
 DISP_ON
 NoConn ~ 5700 2600
-NoConn ~ 3000 4000
-NoConn ~ 3000 3900
-NoConn ~ 3000 3800
+NoConn ~ 5700 3200
+NoConn ~ 5700 3100
+NoConn ~ 5700 3000
 $Comp
 L CONN_2 P2
@@
 F 3 "" H 1550 3400 60  0000 C CNN
 	1    1550 3400
-	-1   0    0    1
+	-1   0    0    -1
 $EndComp
 Wire Wire Line
@@
 VDD
 $Comp
-L GND #PWR28
+L GND #PWR033
 U 1 1 552F45D9
 P 1950 4050
-F 0 "#PWR28" H 1950 4050 30  0001 C CNN
+F 0 "#PWR033" H 1950 4050 30  0001 C CNN
 F 1 "GND" H 1950 3980 30  0001 C CNN
 F 2 "" H 1950 4050 60  0000 C CNN
@@
 Text HLabel 5700 3450 2    60   Input ~ 0
 ACC_INT
+Text Label 2400 3300 0    60   ~ 0
+RX
+Text Label 1900 3500 0    60   ~ 0
+TX
 $EndSCHEMATC
