File: mcu.sch (KiCad schematic (older format))
At the start: 10 parts, among them IC1 BUQ2-ATXMEGA128A4U-A, P2 SERIAL, P3 POWER, U9 TAG-CONNECT-ATMEL-PDI-CONNECT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

Commit message: Some changes?
Connections:
- net BATTERY_SENSE: now reaches IC1.41 (AC1/ADC1/PA1)
- net ACC_INT: no longer names the net of IC1.5 (ADC9/PB1)
Changed lines of the file:
@@
 $Descr A4 11693 8268
 encoding utf-8
-Sheet 8 11
+Sheet 8 10
 Title ""
 Date ""
@@
 $EndDescr
 $Comp
-L BUQ2-ATXMEGA128A4U-A IC1
-U 1 1 54464F09
-P 3900 3500
-F 0 "IC1" H 3150 4700 40  0000 L BNN
-F 1 "BUQ2-ATXMEGA128A4U-A" H 4250 2150 40  0000 L BNN
-F 2 "buq2:BUQ2-TQFP44" H 3900 3500 35  0001 C CIN
-F 3 "" H 3900 3500 60  0000 C CNN
-	1    3900 3500
-	1    0    0    -1
-$EndComp
-$Comp
 L TAG-CONNECT-ATMEL-PDI-CONNECTOR U9
 U 1 1 54464F10
@@
 $EndComp
 $Comp
-L GND #PWR030
+L GND #PWR16
 U 1 1 54464F33
 P 4100 1400
-F 0 "#PWR030" H 4100 1400 30  0001 C CNN
+F 0 "#PWR16" H 4100 1400 30  0001 C CNN
 F 1 "GND" H 4100 1330 30  0001 C CNN
 F 2 "" H 4100 1400 60  0000 C CNN
@@
 NoConn ~ 6100 1450
 $Comp
-L GND #PWR031
+L GND #PWR32
 U 1 1 54464F41
 P 7250 1600
-F 0 "#PWR031" H 7250 1600 30  0001 C CNN
+F 0 "#PWR32" H 7250 1600 30  0001 C CNN
 F 1 "GND" H 7250 1530 30  0001 C CNN
 F 2 "" H 7250 1600 60  0000 C CNN
@@
 $EndComp
 $Comp
-L GND #PWR032
+L GND #PWR13
 U 1 1 54464F47
 P 3900 5100
-F 0 "#PWR032" H 3900 5100 30  0001 C CNN
+F 0 "#PWR13" H 3900 5100 30  0001 C CNN
 F 1 "GND" H 3900 5030 30  0001 C CNN
 F 2 "" H 3900 5100 60  0000 C CNN
@@
 Text HLabel 5700 2700 2    60   Input ~ 0
 DISP_ON
-NoConn ~ 5700 2600
 NoConn ~ 5700 3200
 NoConn ~ 5700 3100
@@
 VDD
 $Comp
-L GND #PWR033
+L GND #PWR1
 U 1 1 552F45D9
 P 1950 4050
-F 0 "#PWR033" H 1950 4050 30  0001 C CNN
+F 0 "#PWR1" H 1950 4050 30  0001 C CNN
 F 1 "GND" H 1950 3980 30  0001 C CNN
 F 2 "" H 1950 4050 60  0000 C CNN
@@
 Text Notes 5600 2200 0    60   ~ 0
 VDD at AREF should make it possible for simple battery monitor
-Text HLabel 5700 3450 2    60   Input ~ 0
-ACC_INT
 Text Label 2400 3300 0    60   ~ 0
 RX
 Text Label 1900 3500 0    60   ~ 0
 TX
+Text HLabel 5700 2600 2    60   Input ~ 0
+BATTERY_SENSE
+$Comp
+L BUQ2-ATXMEGA128A4U-A IC1
+U 1 1 54464F09
+P 3900 3500
+F 0 "IC1" H 3150 4700 40  0000 L BNN
+F 1 "BUQ2-ATXMEGA128A4U-A" H 4250 2150 40  0000 L BNN
+F 2 "buq2:BUQ2-TQFP44" H 3900 3500 35  0001 C CIN
+F 3 "" H 3900 3500 60  0000 C CNN
+	1    3900 3500
+	1    0    0    -1
+$EndComp
+NoConn ~ 5700 3450
 $EndSCHEMATC
